File: BorosDriver.kicad_pcb (KiCad board)
At the start: 2 copper layers, 88.9 x 190.5 mm, 86 parts, among them J1 VIN1, J10 M2B, J11 OUT, J12 T2_PWR, J13 T1_PWR, J14 T2, J15 T1, J2 TRIG_IO, J3 MA_PWR, J4 VIN2, J5 M1A, J6 M2A, J7 MB_PWR, J8 CV_IO, J9 M1B, Q1 MMBT3904, Q2 MMBT3904, Q3 MMBT3904, Q4 MMBT3904, Q5 MMBT3904, Q6 MMBT3904, Q7 MMBT3904, Q8 IRF640N, Q9 IRF640N, SW1 TRIG_I/O, SW2 SW_DIP_x03, SW3 CV_I/O, SW4 PWR, U1 L293D, U2 TEENSY_4.1_MINIMAL, U3 L293D, U4 MCP6002-xSN, U5 PT8211, U6 LM7805_TO220, U7 ClassD_Daughter

Commit message: layout progress
Parts:
- moved J9 23.8 mm to (27.0, 154.8)
- moved J10 23.8 mm to (27.0, 166.7)
- moved J5 23.8 mm to (27.0, 131.0)
- moved J6 23.8 mm to (27.0, 142.9)
- moved J14 11.9 mm to (27.0, 119.1)
- moved J15 11.9 mm to (27.0, 107.2)
- turned C3 to 0 degrees
- turned C7 to 0 degrees
Connections:
- C2 pad 1: VDD -> GND
- C2 pad 2: GND -> VDD
- C4 pad 1: VCC -> GND
- C4 pad 2: GND -> VCC
- Q8 pad 2: Net-(J14-Pad1) -> Net-(J15-Pad1)
- Q9 pad 2: Net-(J15-Pad1) -> Net-(J14-Pad1)
- R18 pad 2: T2 -> T1
- R19 pad 2: T1 -> T2
- R22 pad 2: Net-(J12-Pad1) -> Net-(J13-Pad1)
- R23 pad 2: Net-(J13-Pad1) -> Net-(J12-Pad1)
- R24 pad 2: Net-(J12-Pad1) -> Net-(J13-Pad1)
- R25 pad 2: Net-(J13-Pad1) -> Net-(J12-Pad1)
- U1 pad 1: M1AEN -> M1BEN
- U1 pad 10: M2A1 -> M2B1
- U1 pad 11: Net-(J6-Pad2) -> Net-(J10-Pad2)
- U1 pad 14: Net-(J6-Pad1) -> Net-(J10-Pad1)
- U1 pad 15: M2A2 -> M2B2
- U1 pad 2: M1A2 -> M1B2
- U1 pad 3: Net-(J5-Pad1) -> Net-(J9-Pad1)
- U1 pad 6: Net-(J5-Pad2) -> Net-(J9-Pad2)
- U1 pad 7: M1A1 -> M1B1
- U1 pad 9: M2AEN -> M2BEN
- U2 pad 10: Net-(U2-Pad10) -> M1A1
- U2 pad 11: Net-(U2-Pad11) -> M2A1
- U2 pad 12: Net-(U2-Pad12) -> M2A2
- U2 pad 13: Net-(U2-Pad13) -> M1A2
- U2 pad 14: Net-(U2-Pad14) -> M1AEN
- U2 pad 16: Net-(U2-Pad16) -> T1
- U2 pad 17: Net-(U2-Pad17) -> T2
- U2 pad 2: Net-(U2-Pad2) -> M2BEN
- U2 pad 3: Net-(U2-Pad3) -> M1B1
- U2 pad 4: Net-(U2-Pad4) -> M2B1
- U2 pad 5: Net-(U2-Pad5) -> M2B2
- U2 pad 6: Net-(U2-Pad6) -> M1B2
- U2 pad 7: Net-(U2-Pad7) -> M1BEN
- U2 pad 8: Net-(U2-Pad8) -> M2AEN
- U3 pad 1: M1BEN -> M1AEN
- U3 pad 10: M2B1 -> M2A1
- U3 pad 11: Net-(J10-Pad2) -> Net-(J6-Pad2)
- U3 pad 14: Net-(J10-Pad1) -> Net-(J6-Pad1)
- U3 pad 15: M2B2 -> M2A2
- U3 pad 2: M1B2 -> M1A2
- U3 pad 3: Net-(J9-Pad1) -> Net-(J5-Pad1)
- U3 pad 6: Net-(J9-Pad2) -> Net-(J5-Pad2)
- U3 pad 7: M1B1 -> M1A1
- U3 pad 9: M2BEN -> M2AEN
Routing:
- net M2B1: track 0.00 -> 139.3 mm
- net M2BEN: track 0.00 -> 135.7 mm
- net M2A1: track 0.00 -> 129.9 mm
- net M1B1: track 0.00 -> 129.3 mm
- net M2AEN: track 0.00 -> 124.3 mm
- net M1A1: track 0.00 -> 120.8 mm
- net M2B2: track 0.00 -> 120.4 mm
- net M1B2: track 0.00 -> 113.3 mm
- net M1BEN: track 0.00 -> 113.2 mm
- net M2A2: track 0.00 -> 108.8 mm
- net M1AEN: track 0.00 -> 101.6 mm
- net M1A2: track 0.00 -> 101.5 mm
- net VDD: track 0.00 -> 88.1 mm
- net +5V: track 0.00 -> 84.1 mm, vias 0 -> 4
- net VCC: track 0.00 -> 83.2 mm
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
Commit message: layout finished
Parts:
- J11: footprint HammerheadAudio:JLC-StereoJack-MonoSwitched-C2764616_VAL -> HammerheadAudio:JLC-StereoJack-TRS-C2764616
- moved R10 14.7 mm to (73.8, 115.1)
- moved R13 11.9 mm to (71.8, 115.1), turned to 90 degrees
- moved Q3 6.02 mm to (68.7, 115.1), turned to 180 degrees
- moved Q4 1.19 mm to (55.2, 75.9)
- moved Q5 1.19 mm to (87.7, 75.8)
- moved Q6 1.19 mm to (49.6, 75.8)
- moved Q7 1.19 mm to (82.2, 75.8)
- moved R18 1.19 mm to (59.9, 75.9)
- moved R19 1.19 mm to (92.5, 75.8)
- moved R20 1.19 mm to (57.9, 75.9)
- moved R21 1.19 mm to (90.5, 75.8)
- moved R22 1.19 mm to (52.4, 75.8)
- moved R23 1.19 mm to (84.9, 75.8)
- moved R24 1.19 mm to (46.8, 75.8)
- moved R25 1.19 mm to (79.4, 75.8)
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Connections:
- J3 pad 1: Net-(C3-Pad2) -> Net-(C7-Pad2)
- J3 pad 3: Net-(C3-Pad2) -> Net-(C7-Pad2)
- J3 pad 5: Net-(C3-Pad2) -> Net-(C7-Pad2)
- J7 pad 1: Net-(C7-Pad2) -> Net-(C3-Pad2)
- J7 pad 3: Net-(C7-Pad2) -> Net-(C3-Pad2)
- J7 pad 5: Net-(C7-Pad2) -> Net-(C3-Pad2)
- RV2 pad 2: CTRL1 -> CTRL2
- RV3 pad 2: CTRL2 -> CTRL3
- U2 pad 23: Net-(U2-Pad23) -> UM
- U2 pad 24: Net-(U2-Pad24) -> FAULT
- U2 pad 26: Net-(U2-Pad26) -> MUTE_IN
- U2 pad 27: Net-(U2-Pad27) -> DIP3
- U2 pad 28: Net-(U2-Pad28) -> DIP1
- U2 pad 29: Net-(U2-Pad29) -> CV_OUT
- U2 pad 30: Net-(U2-Pad30) -> CV_IN
- U2 pad 31: Net-(U2-Pad31) -> DIP2
- U2 pad 32: Net-(U2-Pad32) -> CLK_IN
- U2 pad 33: Net-(U2-Pad33) -> CTRL1
- U2 pad 34: Net-(U2-Pad34) -> GND
- U2 pad 35: Net-(U2-Pad35) -> CTRL2
- U2 pad 36: Net-(U2-Pad36) -> CTRL3
- U2 pad 37: Net-(U2-Pad37) -> VOL
- U2 pad 40: Net-(U2-Pad40) -> TRIG_OUT
Routing:
- net +5V: track 84.1 -> 609.9 mm, vias 4 -> 6
- net Net-(J12-Pad1): track 0.00 -> 309.0 mm, vias 0 -> 15
- net Net-(J13-Pad1): track 0.00 -> 215.3 mm, vias 0 -> 15
- net Net-(C3-Pad2): track 0.00 -> 213.5 mm
- net AR: track 0.00 -> 210.9 mm, vias 0 -> 1
- net Net-(C7-Pad2): track 0.00 -> 204.7 mm
- net AL: track 0.00 -> 200.9 mm, vias 0 -> 1
- net VDD: track 88.1 -> 256.6 mm
- net Net-(J14-Pad1): track 0.00 -> 87.9 mm
- net +3V3: track 5.04 -> 91.0 mm
- net Net-(Q1-Pad2): track 0.00 -> 81.4 mm
- net FAULT: track 0.00 -> 76.1 mm
- net Net-(R11-Pad2): track 0.00 -> 76.0 mm
- net UM: track 0.00 -> 75.5 mm
- net Net-(R4-Pad2): track 0.00 -> 69.8 mm
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