File: BorosDriver.sch (KiCad schematic (older format))
At the start: 85 parts, among them J1 VIN1, J10 M2B, J11 OUT, J12 T2_PWR, J13 T1_PWR, J14 T2, J15 T1, J2 TRIG_IO, J3 MA_PWR, J4 VIN2, J5 M1A, J6 M2A, J7 MB_PWR, J8 CV_IO, J9 M1B, Q1 MMBT3904, Q2 MMBT3904, Q3 MMBT3904, Q4 MMBT3904, Q5 MMBT3904, Q6 MMBT3904, Q7 MMBT3904, Q8 IRF640N, Q9 IRF640N, SW1 TRIG_I/O, SW2 SW_DIP_x03, SW3 CV_I/O, SW4 PWR, U1 L293D, U2 TEENSY_4.1_MINIMAL, U3 L293D, U4 MCP6002-xSN, U5 PT8211, U6 LM7805_TO220, U7 ClassD_Daughter

Commit message: layout progress
Connections:
- net GND: now also C2.1, C4.1; no longer C2.2, C4.2
- net M1A1: now also U2.10 (8_PWM), U3.7 (2A); no longer U1.7 (2A)
- net M1A2: now also U2.13 (11_PWM), U3.2 (1A); no longer U1.2 (1A)
- net M1AEN: now also U2.14 (12_PWM), U3.1 (EN1,2); no longer U1.1 (EN1,2)
- net M1B1: now also U1.7 (2A), U2.3 (1_PWM); no longer U3.7 (2A)
- net M1B2: now also U1.2 (1A), U2.6 (4_PWM); no longer U3.2 (1A)
- net M1BEN: now also U1.1 (EN1,2), U2.7 (5_PWM); no longer U3.1 (EN1,2)
- net M2A1: now also U2.11 (9_PWM), U3.10 (3A); no longer U1.10 (3A)
- net M2A2: now also U2.12 (10_PWM), U3.15 (4A); no longer U1.15 (4A)
- net M2AEN: now also U2.8 (6_PWM), U3.9 (EN3,4); no longer U1.9 (EN3,4)
- net M2B1: now also U1.10 (3A), U2.4 (2_PWM); no longer U3.10 (3A)
- net M2B2: now also U1.15 (4A), U2.5 (3_PWM); no longer U3.15 (4A)
- net M2BEN: now also U1.9 (EN3,4), U2.2 (0_PWM); no longer U3.9 (EN3,4)
- net T1: now also R18.2, U2.16 (24_PWM_A10); no longer R19.2
- net T2: now also R19.2, U2.17 (25_PWM_A11); no longer R18.2
- net VCC: now also C4.2; no longer C4.1
- net VDD: now also C2.2; no longer C2.1
- net at J12.1 (Pin_1), J12.3 (Pin_3), J12.5 (Pin_5)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: now also R23.2, R25.2; no longer R22.2, R24.2
- net at Q8.2 (D): now also J15.1 (Pin_1); no longer J14.1 (Pin_1)
- net at U1.11 (3Y): now also J10.2 (Pin_2); no longer J6.2 (Pin_2)
- net at U1.14 (4Y): now also J10.1 (Pin_1); no longer J6.1 (Pin_1)
- net at U1.3 (1Y): now also J9.1 (Pin_1); no longer J5.1 (Pin_1)
- net at U1.6 (2Y): now also J9.2 (Pin_2); no longer J5.2 (Pin_2)
- net at U3.11 (3Y): now also J6.2 (Pin_2); no longer J10.2 (Pin_2)
- net at U3.14 (4Y): now also J6.1 (Pin_1); no longer J10.1 (Pin_1)
- net at U3.3 (1Y): now also J5.1 (Pin_1); no longer J9.1 (Pin_1)
- net at U3.6 (2Y): now also J5.2 (Pin_2); no longer J9.2 (Pin_2)
- net at Q9.2 (D): now also J14.1 (Pin_1); no longer J15.1 (Pin_1)
- net at J13.1 (Pin_1), J13.3 (Pin_3), J13.5 (Pin_5)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: now also R22.2, R24.2; no longer R23.2, R25.2
- no-connect marks 13 -> 14
Other:
- moved on the sheet: J10, J5, J6, J9, Q4, Q5, Q6, Q7, Q8, Q9, R18, R19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

Commit message: layout finished
Parts:
- J11: footprint HammerheadAudio:JLC-StereoJack-MonoSwitched-C2764616_VAL -> HammerheadAudio:JLC-StereoJack-TRS-C2764616
Connections:
- net CLK_IN: now also U2.32 (40_A16)
- net CTRL1: now also U2.33 (41_A17); no longer RV2.2
- net CTRL2: now also RV2.2, U2.35 (13_LED); no longer RV3.2
- net CV_IN: now also U2.30 (38_A14)
- net CV_OUT: now also U2.29 (37_PWM)
- net DIP1: now also U2.28 (36_PWM)
- net DIP2: now also U2.31 (39_A15)
- net DIP3: now also U2.27 (35)
- net FAULT: now also U2.24 (32)
- net GND: now also U2.34 (GND)
- net MUTE_IN: now also U2.26 (34)
- net TRIG_OUT: now also U2.40 (18_PWM_A4)
- net UM: now also U2.23 (31)
- net VOL: now also U2.37 (15_PWM_A1)
- net CTRL3: now reaches U2.36 (14_PWM_A0)
- net CTRL3: now also RV3.2
- net at J3.1 (Pin_1), J3.3 (Pin_3), J3.5 (Pin_5): now also C7.2, U3.8 (VCC2); no longer C3.2, U1.8 (VCC2)
- net at J7.1 (Pin_1), J7.3 (Pin_3), J7.5 (Pin_5): now also C3.2, U1.8 (VCC2); no longer C7.2, U3.8 (VCC2)
- no-connect marks 14 -> 25
Other:
- moved on the sheet: J11, J3, J7, R17
